Commit message: lidar working in gz

File: urdf/smb_lidar_mount.urdf.xacro (robot description, xacro)
@@ -2,4 +2,5 @@
 <!-- This file contains plugins to simulate an Imu sensor attached to the robot. -->
 <!-- Documentation can be found at http://wiki.ros.org/hector_gazebo_plugins -->
+<!-- <xacro:property name="description_path" value="$(find smb)/description"/> -->
 <robot name="smb" xmlns:xacro="http://www.ros.org/wiki/xacro">
   <xacro:macro name="lidar_mount" params="base_link">
@@ -11,5 +12,5 @@
       <visual>
         <geometry>
-          <mesh filename="package://smb_description/urdf/new_payload/meshes/LidarBoxV2.dae"/>
+          <mesh filename="${description_path}/urdf/new_payload/meshes/LidarBoxV2.dae"/>
         </geometry>
       </visual>
