Commit message: sensors have issues, but robot can be controlled

File: urdf/robot.urdf.xacro (robot description, xacro)
@@ -3,7 +3,7 @@
     <xacro:arg name="use_ros2_control" default="true"/>
     <xacro:arg name="sim_mode" default="true"/>
-    <xacro:include filename="/home/perfrivik/rss_ws/src/smb/description/urdf/smb_standalone.urdf.xacro" />
+    <xacro:include filename="/home/perfrivik/rss_ws/src/smb_description/urdf/smb_standalone.urdf.xacro" />
     <!-- <xacro:if value="$(arg use_ros2_control)"> -->
-    <xacro:include filename="/home/perfrivik/rss_ws/src/smb/description/ros2_control.xacro" />
+    <!-- <xacro:include filename="/home/perfrivik/rss_ws/src/smb/description/ros2_control.xacro" /> -->
     <!-- </xacro:if> -->
     <!-- <xacro:unless value="$(arg use_ros2_control)">

File: urdf/sensor_plugins/smb_lidar.gazebo.xacro (robot description, xacro)
@@ -36,32 +36,34 @@
         </plugin>
       </gazebo>
-      <gazebo reference="rslidar" >
+      <gazebo reference="rslidar">
         <sensor name="rslidar" type="gpu_lidar">
-          <gz_frame_id>rslidar</gz_frame_id>
           <topic>scan</topic>
           <update_rate>10</update_rate>
-          <lidar>
+          <ray>
             <scan>
+              <!-- Horizontal (360-degree rotation for full field of view) -->
               <horizontal>
-                <samples>440</samples>
+                <samples>180</samples> <!-- Higher sample count for denser scan -->
                 <resolution>1</resolution>
-                <min_angle>-3.14</min_angle>
-                <max_angle>3.14</max_angle>
+                <min_angle>-3.14159</min_angle> <!-- -180 degrees -->
+                <max_angle>3.14159</max_angle>  <!-- 180 degrees -->
               </horizontal>
+              <!-- Vertical configuration with 32 channels -->
               <vertical>
-                <samples>440</samples>
+                <samples>32</samples> <!-- RS32 has 32 channels -->
                 <resolution>1</resolution>
-                <min_angle>-${15.0*M_PI/180.0}</min_angle>
-                <max_angle> ${15.0*M_PI/180.0}</max_angle>
+                <min_angle>-0.261799</min_angle> <!-- Approximately -15 degrees in radians -->
+                <max_angle>0.261799</max_angle>  <!-- Approximately +15 degrees in radians -->
               </vertical>
             </scan>
+            <!-- Range settings for RS32 -->
             <range>
-              <min>0.2</min>
-              <max>70.0</max>
-              <resolution>0.01</resolution>
+              <min>0.2</min> <!-- Minimum detection range -->
+              <max>120.0</max> <!-- Maximum detection range; can vary slightly with RS32 models -->
+              <resolution>0.01</resolution> <!-- Resolution of 1 cm for high accuracy -->
             </range>
-            <frame_id>/rslidar</frame_id>
-          </lidar>
-          <alwaysOn>ture</alwaysOn>
+          </ray>
+          <!-- Visualization for Gazebo UI -->
+          <always_on>1</always_on>
           <visualize>true</visualize>
         </sensor>

File: urdf/smb.urdf.xacro (robot description, xacro)
@@ -21,5 +21,18 @@
             <limit effort="100" velocity="10"/>
             <joint_properties damping="0.2" friction="0.2"/>
+            <!-- <gazebo>
+                <plugin filename="gz-sim-joint-controller-system" name="gz::sim::systems::JointController">
+                    <joint_name>${prefix}_WHEEL_JOINT</joint_name>
+                    <initial_velocity>1.0</initial_velocity>
+                </plugin>
+            </gazebo> -->
         </joint>
+        <gazebo>
+            <plugin filename="gz-sim-joint-controller-system" name="gz::sim::systems::JointController">
+                <joint_name>${prefix}_WHEEL_JOINT</joint_name>
+                <!-- <topic> -->
+                <!-- <initial_velocity>0.0</initial_velocity> -->
+            </plugin>
+        </gazebo>
         <link name="${prefix}_WHEEL">
             <collision>
@@ -77,5 +90,5 @@
                 <origin xyz="0 0 0" rpy="0 0 0"/>
                 <geometry>
-                    <box size="$0.1 0.1 0.1"/>
+                    <box size="0.1 0.1 0.1"/>
                 </geometry>
                 <material name="base_material">
@@ -150,4 +163,5 @@
             <origin xyz="0.29082 -0.04542 ${0.0955 + chassisHeight/2.0}" rpy="0 0 0" />
         </xacro:rgb_camera_cam>
+        <!-- LIDAR IS FUCKED -->
         <xacro:if value="${lidar}">
             <xacro:lidar_mount base_link="${base_link_name}"/>

File: urdf/smb_standalone.urdf.xacro (robot description, xacro)
@@ -2,6 +2,6 @@
 <robot xmlns:xacro="http://www.ros.org/wiki/xacro" name="smb">
   <!-- Arguments -->
-  <xacro:arg name="wheel_joint_type"          default="fixed"/> <!-- continuous for gazebo -->
-  <xacro:arg name="simulation"                default="false"/>
+  <xacro:arg name="wheel_joint_type"          default="continuous"/> <!-- continuous for gazebo -->
+  <xacro:arg name="simulation"                default="true"/>
   <xacro:arg name="use_ros_control"           default="false"/>
   <xacro:arg name="lidar"                     default="true"/>
@@ -13,9 +13,10 @@
   <!-- Includes -->
   <!-- This loads a bunch of xacro properties -->
-  <xacro:include filename="$(find smb_description)/urdf/smb_big_properties.urdf.xacro" />
+  <xacro:include filename="smb_big_properties.urdf.xacro" />
   <!-- <xacro:if value="$(arg simulation)">
     <xacro:include filename="$(find smb_description)/urdf/smb_gazebo_addins.urdf.xacro"/>
   </xacro:if> -->
-  <xacro:include filename="$(find smb_description)/urdf/smb.urdf.xacro" />
-  <!-- <xacro:smb wheel_joint_type="$(arg wheel_joint_type)" simulation="$(arg simulation)" tracking_camera="$(arg tracking_camera)"/> -->
+  <xacro:include filename="smb.urdf.xacro" />
+  <!-- Terrible bug here, check the input parameters for the smb!!! do not match I think -->
+  <xacro:smb wheel_joint_type="$(arg wheel_joint_type)" simulation="$(arg simulation)" tracking_camera="$(arg tracking_camera)"/>
 </robot>
