Commit message: lidar works

File: urdf/new_sensor_plugins/smb_lidar.gazebo.xacro (robot description, xacro)
@@ -5,4 +5,5 @@
   <xacro:arg name="pointcloud_topic"	default="/rslidar/points"/>
   <xacro:property name="gpu" 		value="$(arg gpu)" />
+  <xacro:property name="M_PI" value="3.1415926535897931" />
   <xacro:macro name="LIDAR" params="parent_link simulation">
     <xacro:if value="${simulation}">
@@ -35,13 +36,13 @@
         </plugin>
       </gazebo>
-      <gazebo reference="base_link" >
-        <sensor name="base_link" type="gpu_lidar">
-          <gz_frame_id>base_link</gz_frame_id>
+      <gazebo reference="rslidar" >
+        <sensor name="rslidar" type="gpu_lidar">
+          <gz_frame_id>rslidar</gz_frame_id>
           <topic>scan</topic>
-          <update_rate>30</update_rate>
+          <update_rate>10</update_rate>
           <lidar>
             <scan>
               <horizontal>
-                <samples>2800</samples>
+                <samples>440</samples>
                 <resolution>1</resolution>
                 <min_angle>-3.14</min_angle>
@@ -49,16 +50,16 @@
               </horizontal>
               <vertical>
-                <samples>1</samples>
-                <resolution>0.1</resolution>
-                <min_angle>0.0</min_angle>
-                <max_angle>0.0</max_angle>
+                <samples>440</samples>
+                <resolution>1</resolution>
+                <min_angle>-${15.0*M_PI/180.0}</min_angle>
+                <max_angle> ${15.0*M_PI/180.0}</max_angle>
               </vertical>
             </scan>
             <range>
               <min>0.2</min>
-              <max>30.0</max>
+              <max>70.0</max>
               <resolution>0.01</resolution>
             </range>
-            <frame_id>/base_link</frame_id>
+            <frame_id>/rslidar</frame_id>
           </lidar>
           <alwaysOn>ture</alwaysOn>
