Commit message: rgb and depth camera

File: urdf/new_sensor_plugins/smb_rgb_camera.gazebo.xacro (robot description, xacro)
@@ -4,11 +4,47 @@
     <xacro:property name="camera_topic" value="/${name}/image_raw" />
     <xacro:property name="camera_info_topic" value="/${name}/camera_info" />
+    <!-- <gazebo> -->
+          <!-- <plugin
+      filename="gz-sim-physics-system"
+      name="gz::sim::systems::Physics">
+    </plugin> -->
+    <!-- <plugin
+      filename="gz-sim-sensors-system"
+      name="gz::sim::systems::Sensors">
+      <render_engine>ogre2</render_engine>
+    </plugin> -->
+    <!-- <plugin
+      filename="gz-sim-user-commands-system"
+      name="gz::sim::systems::UserCommands">
+    </plugin>
+    <plugin
+      filename="gz-sim-scene-broadcaster-system"
+      name="gz::sim::systems::SceneBroadcaster">
+    </plugin> -->
+    <!-- </gazebo> -->
     <gazebo reference="${link_name}">
-      <sensor type="camera" name="${name}">
+        <sensor name="camera" type="camera">
+          <camera>
+            <horizontal_fov>1.047</horizontal_fov>
+            <image>
+              <width>320</width>
+              <height>240</height>
+            </image>
+            <clip>
+              <near>0.1</near>
+              <far>100</far>
+            </clip>
+          </camera>
+          <always_on>1</always_on>
+          <update_rate>30</update_rate>
+          <visualize>true</visualize>
+          <topic>camera</topic>
+        </sensor>
+      <!-- <sensor type="camera" name="${name}">
         <pose>0.0066 0 0 0 0 0</pose>
         <visualize>false</visualize>
         <update_rate>${rate}</update_rate>
         <camera>
-          <horizontal_fov>1.192</horizontal_fov> <!-- 80 deg-->
+          <horizontal_fov>1.192</horizontal_fov>
           <image>
             <width>1440</width>
@@ -40,5 +76,5 @@
           <distortionT2>0.0</distortionT2>
         </plugin>
-      </sensor>
+      </sensor> -->
     </gazebo>
   </xacro:macro>

File: urdf/new_sensor_plugins/smb_rgb_camera.urdf.xacro (robot description, xacro)
@@ -4,5 +4,5 @@
 <robot name="smb" xmlns:xacro="http://www.ros.org/wiki/xacro">
   <!-- INCLUDE PLUGIN -->
-  <xacro:include filename="$(find smb_description)/urdf/sensor_plugins/smb_rgb_camera.gazebo.xacro"/>
+  <xacro:include filename="$(find smb_description)/urdf/new_sensor_plugins/smb_rgb_camera.gazebo.xacro"/>
   <xacro:macro name="rgb_camera_cam" params="*origin id base_link simulation">
     <!--                              Camera  Properties 				          	-->
@@ -19,10 +19,10 @@
       <visual>
         <geometry>
-          <mesh filename="package://smb_description/urdf/new_payload/meshes/SMB_blackfly_camera.dae"/>
+          <mesh filename="${description_path}/urdf/new_payload/meshes/SMB_blackfly_camera.dae"/>
         </geometry>
       </visual>
       <collision>
         <geometry>
-          <mesh filename="package://smb_description/urdf/new_payload/meshes/SMB_blackfly_camera.dae"/>
+          <mesh filename="${description_path}/urdf/new_payload/meshes/SMB_blackfly_camera.dae"/>
         </geometry>
       </collision>
@@ -49,7 +49,7 @@
       <child link="rgb_camera${id}_optical_link"/>
     </joint>
-    <xacro:if value="${simulation}">
-        <xacro:rgb_camera_camera_plugin name="rgb_camera" link_name="${rgb_camera_link}" rate="${rgb_camera_update_rate}"/>
-    </xacro:if>
+    <!-- <xacro:if value="${simulation}"> -->
+    <xacro:rgb_camera_camera_plugin name="rgb_camera" link_name="${rgb_camera_link}" rate="${rgb_camera_update_rate}"/>
+    <!-- </xacro:if> -->
   </xacro:macro>
 </robot>

File: urdf/smb_rgb_camera.urdf.xacro (robot description, xacro)
@@ -4,5 +4,5 @@
 <robot name="smb" xmlns:xacro="http://www.ros.org/wiki/xacro">
   <!-- INCLUDE PLUGIN -->
-  <xacro:include filename="$(find smb_description)/urdf/sensor_plugins/smb_rgb_camera.gazebo.xacro"/>
+  <xacro:include filename="$(find smb_description)/urdf/new_sensor_plugins/smb_rgb_camera.gazebo.xacro"/>
   <xacro:macro name="rgb_camera_cam" params="*origin id base_link simulation">
     <!--                              Camera  Properties 				          	-->
@@ -31,7 +31,7 @@
         </material>
     </link>
-      <gazebo reference="${rgb_camera_link}">
-        <material>Gazebo/Red</material>
-      </gazebo>
+    <gazebo reference="${rgb_camera_link}">
+      <material>Gazebo/Red</material>
+    </gazebo>
     <joint name="rgb_camera${id}_camera_joint" type="fixed">
       <!-- <origin xyz="${rgb_camera_origin_xyz}" rpy="${rgb_camera_origin_rpy}"/> -->
