Commit message: description cleanup

File: urdf/sensor_plugins/smb_imu.gazebo.xacro (robot description, xacro)
@@ -12,4 +12,9 @@
     <xacro:property name="imu_topic" value="/imu"/>
     <xacro:if value="${simulation}">
+    <gazebo>
+        <plugin filename="gz-sim-imu-system"
+            name="gz::sim::systems::Imu">
+        </plugin>
+    </gazebo>
     <gazebo reference="${imu_link}">
       <sensor name="imu_sensor" type="imu">
@@ -17,5 +22,6 @@
         <update_rate>${imu_update_rate}</update_rate>
         <visualize>true</visualize>
-        <plugin name="smb_imu_plugin" filename="libgazebo_ros_imu_sensor.so">
+        <topic>/imu</topic>
+        <!-- <plugin name="smb_imu_plugin" filename="libgazebo_ros_imu_sensor.so">
           <ros>
             <namespace>/</namespace>
@@ -23,5 +29,5 @@
           </ros>
           <initial_orientation_as_reference>false</initial_orientation_as_reference>
-        </plugin>
+        </plugin> -->
       </sensor>
     </gazebo>
@@ -42,5 +48,5 @@
         <origin rpy="0 0 0" xyz="0 0 0"/>
         <geometry>
-          <mesh filename="${description_path}/urdf/new_payload/meshes/SMB_imu.dae"/>
+          <mesh filename="${description_path}/urdf/meshes/SMB_imu.dae"/>
         </geometry>
       </visual>
@@ -48,5 +54,5 @@
         <origin rpy="0 0 0" xyz="0 0 0"/>
         <geometry>
-          <mesh filename="${description_path}/urdf/new_payload/meshes/SMB_imu.dae"/>
+          <mesh filename="${description_path}/urdf/meshes/SMB_imu.dae"/>
         </geometry>
       </collision>

File: urdf/sensor_plugins/smb_odometry.gazebo.xacro (robot description, xacro)
@@ -2,6 +2,22 @@
 <robot xmlns:xacro="http://www.ros.org/wiki/xacro" name="smb">
 <xacro:macro name="odometry_plugin" params="sensor_link topic_name odom_frame:=camera_odom_frame child_odom_frame:=camera_pose_frame publish_tf:=true rate:=20 max_linear_speed_before_settle:=0.001 max_angular_speed_before_settle:=0.001">
-    <gazebo>
-        <plugin name="smb_odometry_plugin" filename="libodometry_source_plugin.so">
+    <gazebo reference="tracking_camera_link">
+           <sensor name="depth_camera1" type="depth_camera">
+          <update_rate>10</update_rate>
+          <topic>depth_camera</topic>
+          <camera>
+            <horizontal_fov>1.05</horizontal_fov>
+            <image>
+              <width>256</width>
+              <height>256</height>
+              <format>R_FLOAT32</format>
+            </image>
+            <clip>
+              <near>0.1</near>
+              <far>10.0</far>
+            </clip>
+          </camera>
+          </sensor>
+        <!-- <plugin name="smb_odometry_plugin" filename="libodometry_source_plugin.so">
             <robotNamespace>smb</robotNamespace>
             <bodyName>${sensor_link}</bodyName>
@@ -16,5 +32,5 @@
             <maxLinearSpeedBeforeSettle>${max_linear_speed_before_settle}</maxLinearSpeedBeforeSettle>
             <maxAngularSpeedBeforeSettle>${max_angular_speed_before_settle}</maxAngularSpeedBeforeSettle>
-        </plugin>
+        </plugin> -->
     </gazebo>
 </xacro:macro>

File: urdf/sensor_plugins/smb_odometry.urdf.xacro (robot description, xacro)
@@ -7,10 +7,4 @@
   <xacro:property name="realsense_t265_width"  value="0.013"/>
   <xacro:property name="realsense_t265_housing_center_x_offset"  value="0.00910"/>
-  <!-- t265_origin_xyz is the offset to the parent link -->
-  <!-- t265_origin_rpy is the fixed axis roll, pitch and yaw angle such that the resulting frame has
-       the x axis pointing forward ("out of camera"),
-       the y axis pointing left and the z axis pointing upward -->
-  <!-- another frame "realsense_t265_odom_frame is created that is in line with the one documented here:
-       https://www.intel.com/content/dam/support/us/en/documents/emerging-technologies/intel-realsense-technology/IntelRealSenseTrackingT265Datasheet.pdf -->
   <xacro:macro name="REALSENSE_T265" params="base_link t265_origin_xyz t265_origin_rpy simulation">
     <link name="tracking_camera_link">
@@ -68,7 +62,7 @@
     </joint>
     -->
-    <xacro:if value="${simulation}">
-          <xacro:odometry_plugin sensor_link="tracking_camera_link" topic_name="/tracking_camera/odom/sample" odom_frame="tracking_camera_odom_frame" child_odom_frame="tracking_camera_pose_frame" rate="200" max_linear_speed_before_settle="0.01" max_angular_speed_before_settle="0.05" publish_tf="false"/>
-    </xacro:if>
+    <!-- <xacro:if value="${simulation}"> -->
+    <xacro:odometry_plugin sensor_link="tracking_camera_link" topic_name="/tracking_camera/odom/sample" odom_frame="tracking_camera_odom_frame" child_odom_frame="tracking_camera_pose_frame" rate="200" max_linear_speed_before_settle="0.01" max_angular_speed_before_settle="0.05" publish_tf="false"/>
+    <!-- </xacro:if> -->
   </xacro:macro>
 </robot>

File: urdf/sensor_plugins/smb_rgb_camera.urdf.xacro (robot description, xacro)
@@ -4,5 +4,5 @@
 <robot name="smb" xmlns:xacro="http://www.ros.org/wiki/xacro">
   <!-- INCLUDE PLUGIN -->
-  <xacro:include filename="$(find smb_description)/urdf/new_sensor_plugins/smb_rgb_camera.gazebo.xacro"/>
+  <xacro:include filename="$(find smb_description)/urdf/sensor_plugins/smb_rgb_camera.gazebo.xacro"/>
   <xacro:macro name="rgb_camera_cam" params="*origin id base_link simulation">
     <!--                              Camera  Properties 				          	-->
@@ -19,10 +19,10 @@
       <visual>
         <geometry>
-          <mesh filename="${description_path}/urdf/new_payload/meshes/SMB_blackfly_camera.dae"/>
+          <mesh filename="${description_path}/urdf/meshes/SMB_blackfly_camera.dae"/>
         </geometry>
       </visual>
       <collision>
         <geometry>
-          <mesh filename="${description_path}/urdf/new_payload/meshes/SMB_blackfly_camera.dae"/>
+          <mesh filename="${description_path}/urdf/meshes/SMB_blackfly_camera.dae"/>
         </geometry>
       </collision>

File: urdf/smb.urdf.xacro (robot description, xacro)
@@ -2,24 +2,13 @@
 <robot xmlns:xacro="http://www.ros.org/wiki/xacro" name="smb">
     <!-- TODO: replace this arg by other ones like sensors, legacy, etc -->
+    <xacro:property name="description_path" value="$(find smb_description)"/>
     <xacro:arg name="lidar" default="true"/>
-    <xacro:arg name="tracking_camera" default="false"/>
-    <!-- Defines colors and calculates typical inertias -->
-    <xacro:include filename="$(find smb_description)/urdf/smb_utils.urdf.xacro" />
-    <!-- Defines IMU macro -->
-    <xacro:include filename="$(find smb_description)/urdf/sensor_plugins/smb_imu.gazebo.xacro"/>
-    <!-- Defines Lidar macro -->
-    <xacro:if value="$(arg lidar)">
-        <xacro:include filename="$(find smb_description)/urdf/sensor_plugins/smb_robosense.gazebo.xacro"/>
-    </xacro:if>
-    <!-- Defines odometry macro -->
-    <xacro:include filename="$(find smb_description)/urdf/sensor_plugins/smb_odometry.gazebo.xacro"/>
-    <!-- Defines realsense_t265 (tracking camera) macro -->
-    <xacro:if value="$(arg tracking_camera)">
-        <xacro:include filename="$(find smb_description)/urdf/realsense_t265.urdf.xacro"/>
-    </xacro:if>
-    <!-- Defines blackfly rgb_camera camera macro -->
-    <xacro:include filename="$(find smb_description)/urdf/smb_rgb_camera.urdf.xacro"/>
-    <!-- Defines lidar macro -->
-    <xacro:include filename="$(find smb_description)/urdf/smb_lidar_mount.urdf.xacro"/>
+    <xacro:arg name="tracking_camera" default="true"/>
+    <xacro:include filename="${description_path}/urdf/smb_utils.urdf.xacro" />
+    <xacro:include filename="${description_path}/urdf/sensor_plugins/smb_imu.gazebo.xacro"/>
+    <xacro:include filename="${description_path}/urdf/sensor_plugins/smb_lidar.gazebo.xacro"/>
+    <xacro:include filename="${description_path}/urdf/sensor_plugins/smb_odometry.urdf.xacro"/>
+    <xacro:include filename="${description_path}/urdf/sensor_plugins/smb_rgb_camera.urdf.xacro"/>
+    <xacro:include filename="${description_path}/urdf/smb_lidar_mount.urdf.xacro"/>
     <!-- Model macros -->
     <xacro:macro name="wheel" params="prefix X Y wheel_joint_type friction_coeff:=0.2 transmission_reduction:=${wheelTransmission}" >
@@ -43,5 +32,5 @@
                 <origin xyz="0 0 0" rpy="1.570796 0  0" />
                 <geometry>
-                    <mesh filename="package://smb_description/urdf/meshes/wheel.dae" />
+                    <mesh filename="${description_path}/urdf/meshes/wheel.dae"/>
                 </geometry>
             </visual>
@@ -52,28 +41,4 @@
             </inertial>
         </link>
-        <gazebo reference="${prefix}_WHEEL">
-            <mu1 value="${friction_coeff}"/>
-            <mu2 value="${friction_coeff}"/>
-            <fdir1 value="1 0 0"/>
-            <kp>10000000.0</kp>
-            <kd>1.0</kd>
-            <minDepth>0.005</minDepth>
-            <maxVel>100.0</maxVel>
-            <material>Gazebo/DarkGrey</material>
-        </gazebo>
-        <transmission name="${prefix}_WHEEL_TRANS">
-            <type>transmission_interface/SimpleTransmission</type>
-            <joint name="${prefix}_WHEEL_JOINT">
-                <hardwareInterface>hardware_interface/VelocityJointInterface</hardwareInterface>
-                <hardwareInterface>hardware_interface/EffortJointInterface</hardwareInterface>
-                <hardwareInterface>hardware_interface/PositionJointInterface</hardwareInterface>
-            </joint>
-            <actuator name="${prefix}_WHEEL_ACTUATOR">
-                <hardwareInterface>hardware_interface/VelocityJointInterface</hardwareInterface>
-                <hardwareInterface>hardware_interface/EffortJointInterface</hardwareInterface>
-                <hardwareInterface>hardware_interface/PositionJointInterface</hardwareInterface>
-                <mechanicalReduction>${transmission_reduction}</mechanicalReduction>
-            </actuator>
-        </transmission>
     </xacro:macro>
     <xacro:macro name="chassis">
@@ -123,6 +88,5 @@
                 <origin xyz="${topXOffset} 0 0" rpy="0 0 0"/>
                 <geometry>
-                    <!-- <box size="${topLength} ${topWidth} ${topHeight}"/> -->
-                     <mesh filename="package://smb_description/urdf/new_payload/meshes/SMB_step.dae"/>
+                    <mesh filename="${description_path}/urdf/meshes/SMB_step.dae"/>
                 </geometry>
             </collision>
@@ -130,6 +94,5 @@
                 <origin xyz="0 0 0" rpy="0 0 0"/>
                 <geometry>
-                    <!-- <box size="${topLength} ${topWidth} ${topHeight}"/> -->
-                     <mesh filename="package://smb_description/urdf/new_payload/meshes/SMB_step.dae"/>
+                    <mesh filename="${description_path}/urdf/meshes/SMB_step.dae"/>
                 </geometry>
             </visual>
@@ -183,7 +146,6 @@
             wheel_joint_type="${wheel_joint_type}"
             friction_coeff="0.7"/>
-        <!-- <xacro:IMU base_link="${base_link_name}" simulation="${simulation}"/> -->
-        <!-- <xacro:GPS base_link="${base_link_name}" simulation="${simulation}"/> -->
-        <!-- <xacro:rgb_camera_cam id="" base_link="${base_link_name}" simulation="${simulation}">
+        <xacro:IMU base_link="${base_link_name}" simulation="${simulation}"/>
+        <xacro:rgb_camera_cam id="" base_link="${base_link_name}" simulation="${simulation}">
             <origin xyz="0.29082 -0.04542 ${0.0955 + chassisHeight/2.0}" rpy="0 0 0" />
         </xacro:rgb_camera_cam>
@@ -196,6 +158,6 @@
                 t265_origin_xyz="0.309 0.008 0.352"
                 t265_origin_rpy="0 0 0"
-                simulation="${simulation}"/>
-        </xacro:if> -->
+                simulation="True"/>
+        </xacro:if>
     </xacro:macro>
 </robot>

File: urdf/smb_lidar_mount.urdf.xacro (robot description, xacro)
@@ -12,5 +12,5 @@
       <visual>
         <geometry>
-          <mesh filename="${description_path}/urdf/new_payload/meshes/LidarBoxV2.dae"/>
+          <mesh filename="${description_path}/urdf/meshes/LidarBoxV2.dae"/>
         </geometry>
       </visual>

File: urdf/smb_rgb_camera.urdf.xacro (robot description, xacro)
@@ -4,5 +4,5 @@
 <robot name="smb" xmlns:xacro="http://www.ros.org/wiki/xacro">
   <!-- INCLUDE PLUGIN -->
-  <xacro:include filename="$(find smb_description)/urdf/new_sensor_plugins/smb_rgb_camera.gazebo.xacro"/>
+  <xacro:include filename="$(find smb_description)/urdf/sensor_plugins/smb_rgb_camera.gazebo.xacro"/>
   <xacro:macro name="rgb_camera_cam" params="*origin id base_link simulation">
     <!--                              Camera  Properties 				          	-->
@@ -19,10 +19,10 @@
       <visual>
         <geometry>
-          <mesh filename="package://smb_description/urdf/new_payload/meshes/SMB_blackfly_camera.dae"/>
+          <mesh filename="package://smb_description/urdf/meshes/SMB_blackfly_camera.dae"/>
         </geometry>
       </visual>
       <collision>
         <geometry>
-          <mesh filename="package://smb_description/urdf/new_payload/meshes/SMB_blackfly_camera.dae"/>
+          <mesh filename="package://smb_description/urdf/meshes/SMB_blackfly_camera.dae"/>
         </geometry>
       </collision>

Commit message: description loads correct

File: urdf/sensor_plugins/smb_imu.gazebo.xacro (robot description, xacro)
@@ -48,5 +48,5 @@
         <origin rpy="0 0 0" xyz="0 0 0"/>
         <geometry>
-          <mesh filename="${description_path}/urdf/meshes/SMB_imu.dae"/>
+          <mesh filename="file://$(find smb_description)/urdf/meshes/SMB_imu.dae"/>
         </geometry>
       </visual>
@@ -54,5 +54,5 @@
         <origin rpy="0 0 0" xyz="0 0 0"/>
         <geometry>
-          <mesh filename="${description_path}/urdf/meshes/SMB_imu.dae"/>
+          <mesh filename="file://$(find smb_description)/urdf/meshes/SMB_imu.dae"/>
         </geometry>
       </collision>

File: urdf/sensor_plugins/smb_rgb_camera.urdf.xacro (robot description, xacro)
@@ -19,10 +19,10 @@
       <visual>
         <geometry>
-          <mesh filename="${description_path}/urdf/meshes/SMB_blackfly_camera.dae"/>
+          <mesh filename="file://$(find smb_description)/urdf/meshes/SMB_blackfly_camera.dae"/>
         </geometry>
       </visual>
       <collision>
         <geometry>
-          <mesh filename="${description_path}/urdf/meshes/SMB_blackfly_camera.dae"/>
+          <mesh filename="file://$(find smb_description)/urdf/meshes/SMB_blackfly_camera.dae"/>
         </geometry>
       </collision>

File: urdf/smb.urdf.xacro (robot description, xacro)
@@ -5,5 +5,5 @@
 	<xacro:include filename="$(find smb_description)/urdf/smb_properties.urdf.xacro" />
 	<!-- <xacro:include filename="$(find smb_description)/urdf/gps.urdf.xacro" /> -->
-	<xacro:include filename="$(find smb_description)/urdf/robot_gz_diff_drive_plugin.urdf.xacro" />
+	<xacro:include filename="$(find smb_description)/urdf/sensor_plugins/smb_diff_drive_plugin.urdf.xacro" />
     <xacro:include filename="${description_path}/urdf/sensor_plugins/smb_imu.gazebo.xacro"/>
     <xacro:include filename="${description_path}/urdf/sensor_plugins/smb_lidar.gazebo.xacro"/>
@@ -76,4 +76,54 @@
 			</inertial>
 		</link>
+        <joint name="base_footprint_to_base_link" type="fixed">
+            <parent link="${base_link_name}"/>
+            <child link="base_footprint"/>
+            <origin xyz="0 0 0" rpy="0 0 0"/>
+        </joint>
+        <link name="base_footprint">
+            <inertial>
+                <origin xyz="0 0 0" rpy="0 0 0"/>
+                <mass value="0.1"/>
+                <xacro:box_inertia m="${chassisMass}"
+                             x="${chassisLength}"
+                             y="${chassisWidth}"
+                             z="${chassisHeight}"/>
+            </inertial>
+            <visual>
+                <origin xyz="0 0 0" rpy="0 0 0"/>
+                <geometry>
+                    <box size="0.1 0.1 0.1"/>
+                </geometry>
+                <material name="base_material">
+                    <color rgba="0.8 0.0 0.1 1.0"/>
+                </material>
+            </visual>
+        </link>
+        <link name="top">
+            <collision>
+                <origin xyz="${topXOffset} 0 0" rpy="0 0 0"/>
+                <geometry>
+                    <mesh filename="${description_path}/urdf/meshes/SMB_step.dae"/>
+                </geometry>
+            </collision>
+            <visual>
+                <origin xyz="0 0 0" rpy="0 0 0"/>
+                <geometry>
+                    <mesh filename="${description_path}/urdf/meshes/SMB_step.dae"/>
+                </geometry>
+            </visual>
+        </link>
+        <gazebo reference="top">
+            <material>Gazebo/Grey</material>
+        </gazebo>
+        <gazebo reference="${base_link_name}">
+            <material>Gazebo/Red</material>
+        </gazebo>
+    <joint name="top_to_base_link" type="fixed">
+        <parent link="${base_link_name}"/>
+        <child link="top"/>
+        <!-- <origin xyz="${topXOffset/2.0} 0.0 ${chassisHeight/2.0 + topHeight/2.0}" rpy="0 0 0"/> -->
+        <origin xyz="0.0 0.0 ${chassisHeight/2.0}" rpy="0 0 0"/>
+    </joint>
 	</xacro:macro>
     <!-- urdf -->
@@ -83,5 +133,6 @@
 	<xacro:wheel prefix="LH" X="${backWheelX}" reflect="1" friction_coeff="0.85" />
 	<xacro:wheel prefix="RH" X="${backWheelX}" reflect="-1" friction_coeff="0.85" />
-	<xacro:gps x="0.0" y="0.0" z="${chassisHeight/2}" parent="${base_link_name}" />
+	<!-- <xacro:gps x="0.0" y="0.0" z="${chassisHeight/2}" parent="${base_link_name}" /> -->
+    <!-- define simulation -->
     <xacro:IMU base_link="${base_link_name}" simulation="${simulation}"/>
     <xacro:rgb_camera_cam id="" base_link="${base_link_name}" simulation="${simulation}">

File: urdf/smb_lidar_mount.urdf.xacro (robot description, xacro)
@@ -12,5 +12,5 @@
       <visual>
         <geometry>
-          <mesh filename="${description_path}/urdf/meshes/LidarBoxV2.dae"/>
+          <mesh filename="file://$(find smb_description)/urdf/meshes/LidarBoxV2.dae"/>
         </geometry>
       </visual>

File: urdf/smb_properties.urdf.xacro (robot description, xacro)
@@ -22,3 +22,4 @@
     <xacro:property name="wheelMass" value="5"/>
     <xacro:property name="description_path" value="$(find smb_description)"/>
+    <xacro:property name="simulation" value="true"/>
 </robot>

Commit message: prevent joints from collapsing for correct lidar and imu tf transforms

File: urdf/sensor_plugins/smb_imu.gazebo.xacro (robot description, xacro)
@@ -19,15 +19,12 @@
     <gazebo reference="${imu_link}">
       <sensor name="imu_sensor" type="imu">
+        <gz_frame_id>imu_link</gz_frame_id>
+        <!-- <frame>imu</frame>
+        <gz_frame_id>imu</gz_frame_id> -->
+        <!-- <pose relative_to='imu'>0 0 0 0 0 0</pose> -->
         <always_on>true</always_on>
-        <update_rate>${imu_update_rate}</update_rate>
+        <update_rate>400</update_rate>
         <visualize>true</visualize>
         <topic>/imu</topic>
-        <!-- <plugin name="smb_imu_plugin" filename="libgazebo_ros_imu_sensor.so">
-          <ros>
-            <namespace>/</namespace>
-            <remapping>~/out:=${imu_topic}</remapping>
-          </ros>
-          <initial_orientation_as_reference>false</initial_orientation_as_reference>
-        </plugin> -->
       </sensor>
     </gazebo>
@@ -58,5 +55,5 @@
       </collision>
     </link>
-    <link name="imu">
+    <link name="imu_sensor">
       <inertial>
         <mass value="0.001"/>
@@ -68,5 +65,5 @@
       <origin xyz="0 0 0" rpy="0 0 0"/>
       <parent link="${imu_link}"/>
-      <child link="imu"/>
+      <child link="imu_sensor"/>
     </joint>
     <gazebo reference="${imu_link}">

File: urdf/sensor_plugins/smb_lidar.gazebo.xacro (robot description, xacro)
@@ -7,5 +7,5 @@
   <xacro:property name="M_PI" value="3.1415926535897931" />
   <xacro:macro name="LIDAR" params="parent_link simulation">
-    <xacro:if value="${simulation}">
+    <!-- <xacro:if value="${simulation}"> -->
       <!-- Replacing RS-16 with the default Gazebo lidar -->
       <link name="rslidar">
@@ -29,5 +29,10 @@
         <child link="rslidar"/>
         <origin xyz="0.0 0.0 ${lidarBoxHeight+0.039}" rpy="0 0 0"/>
+        <!-- <axis xyz="0 0 1"/> -->
+        <!-- <limit lower="0.0" upper="0.0" effort="0.0" velocity="0.0"/> -->
       </joint>
+    <gazebo reference='${parent_link}_to_rslidar'>
+      <preserveFixedJoint>true</preserveFixedJoint>
+    </gazebo>
       <gazebo>
         <plugin
@@ -38,5 +43,5 @@
       <gazebo reference="rslidar">
         <sensor name="rslidar" type="gpu_lidar">
-          <frame>rslidar</frame>
+          <!-- <frame>rslidar</frame> -->
           <gz_frame_id>rslidar</gz_frame_id>
           <pose relative_to='rslidar'>0 0 0 0 0 0</pose>
@@ -70,5 +75,5 @@
         </sensor>
       </gazebo>
-    </xacro:if>
+    <!-- </xacro:if> -->
   </xacro:macro>
 </robot>

File: urdf/smb.urdf.xacro (robot description, xacro)
@@ -5,5 +5,5 @@
 	<xacro:include filename="$(find smb_description)/urdf/smb_properties.urdf.xacro" />
 	<!-- <xacro:include filename="$(find smb_description)/urdf/gps.urdf.xacro" /> -->
-	<xacro:include filename="$(find smb_description)/urdf/sensor_plugins/smb_diff_drive_plugin.urdf.xacro" />
+	<!-- <xacro:include filename="$(find smb_description)/urdf/sensor_plugins/smb_diff_drive_plugin.urdf.xacro" /> -->
     <xacro:include filename="${description_path}/urdf/sensor_plugins/smb_imu.gazebo.xacro"/>
     <xacro:include filename="${description_path}/urdf/sensor_plugins/smb_lidar.gazebo.xacro"/>
@@ -40,4 +40,15 @@
 			</inertial>
 		</link>
+		<!-- Add joint controller for this wheel -->
+		<gazebo>
+			<plugin filename="gz-sim-joint-controller-system" name="gz::sim::systems::JointController">
+				<joint_name>${prefix}_WHEEL_JOINT</joint_name>
+				<topic>${prefix}_WHEEL_JOINT_velocity_cmd</topic>
+				<!-- <control_type>velocity</control_type> -->
+				<p_gain>0.0</p_gain> <!-- Proportional gain -->
+				<i_gain>0.0</i_gain> <!-- Integral gain -->
+				<d_gain>5.0</d_gain> <!-- Derivative gain -->
+			</plugin>
+		</gazebo>
 	</xacro:macro>
 	<xacro:macro name="chassis">
@@ -146,4 +157,4 @@
         simulation="True"/>
     <!-- plugins -->
-    <xacro:robot_gz_diff_drive_plugin />
+    <!-- <xacro:robot_gz_diff_drive_plugin /> -->
 </robot>

File: urdf/smb_lidar_mount.urdf.xacro (robot description, xacro)
@@ -29,4 +29,7 @@
       <child link="lidar_mount_link"/>
     </joint>
+    <gazebo reference='lidar_mount_joint'>
+      <preserveFixedJoint>true</preserveFixedJoint>
+    </gazebo>
   </xacro:macro>
 </robot>

Commit message: Update IMU and Lidar update rates

File: urdf/sensor_plugins/smb_imu.gazebo.xacro (robot description, xacro)
@@ -8,5 +8,5 @@
     <xacro:property name="imu_origin_rpy" value="0 0 0"/>
     <xacro:property name="imu_origin_xyz" value="0.2554 -0.02397 ${0.081+chassisHeight/2.0}"/>
-    <xacro:property name="imu_update_rate" value="400"/>
+    <xacro:property name="imu_update_rate" value="200"/>
     <xacro:property name="imu_link" value="imu_link"/>
     <xacro:property name="imu_topic" value="/imu"/>
