Commit message: Update IMU and Lidar update rates

File: urdf/sensor_plugins/smb_imu.gazebo.xacro (robot description, xacro)
@@ -8,5 +8,5 @@
     <xacro:property name="imu_origin_rpy" value="0 0 0"/>
     <xacro:property name="imu_origin_xyz" value="0.2554 -0.02397 ${0.081+chassisHeight/2.0}"/>
-    <xacro:property name="imu_update_rate" value="400"/>
+    <xacro:property name="imu_update_rate" value="200"/>
     <xacro:property name="imu_link" value="imu_link"/>
     <xacro:property name="imu_topic" value="/imu"/>

File: urdf/sensor_plugins/smb_lidar.gazebo.xacro (robot description, xacro)
@@ -47,5 +47,5 @@
           <pose relative_to='rslidar'>0 0 0 0 0 0</pose>
           <topic>scan</topic>
-          <update_rate>5</update_rate>
+          <update_rate>10</update_rate>
           <ray>
             <scan>

Commit message: Updated mesh file paths in URDF and XACRO files to use the package:// syntax for better compatibility.

File: urdf/sensor_plugins/smb_imu.gazebo.xacro (robot description, xacro)
@@ -45,5 +45,5 @@
         <origin rpy="0 0 0" xyz="0 0 0"/>
         <geometry>
-          <mesh filename="file://$(find smb_description)/urdf/meshes/SMB_imu.dae"/>
+          <mesh filename="package://smb_description//urdf/meshes/SMB_imu.dae"/>
         </geometry>
       </visual>
@@ -51,5 +51,5 @@
         <origin rpy="0 0 0" xyz="0 0 0"/>
         <geometry>
-          <mesh filename="file://$(find smb_description)/urdf/meshes/SMB_imu.dae"/>
+          <mesh filename="package://smb_description//urdf/meshes/SMB_imu.dae"/>
         </geometry>
       </collision>

File: urdf/sensor_plugins/smb_rgb_camera.urdf.xacro (robot description, xacro)
@@ -19,10 +19,10 @@
       <visual>
         <geometry>
-          <mesh filename="file://$(find smb_description)/urdf/meshes/SMB_blackfly_camera.dae"/>
+          <mesh filename="package://smb_description//urdf/meshes/SMB_blackfly_camera.dae"/>
         </geometry>
       </visual>
       <collision>
         <geometry>
-          <mesh filename="file://$(find smb_description)/urdf/meshes/SMB_blackfly_camera.dae"/>
+          <mesh filename="package://smb_description//urdf/meshes/SMB_blackfly_camera.dae"/>
         </geometry>
       </collision>

File: urdf/smb.urdf.xacro (robot description, xacro)
@@ -45,5 +45,5 @@
 				<origin xyz="0 0 0" rpy="${pi/2} 0 0" />
 				<geometry>
-					<mesh filename="file://$(find smb_description)/urdf/meshes/wheel.dae" />
+					<mesh filename="package://smb_description/urdf/meshes/wheel.dae" />
 				</geometry>
 			</visual>
@@ -129,5 +129,5 @@
                 <origin xyz="${topXOffset} 0 0" rpy="0 0 0"/>
                 <geometry>
-                    <mesh filename="file://$(find smb_description)/urdf/meshes/SMB_step.dae"/>
+                    <mesh filename="package://smb_description/urdf/meshes/SMB_step.dae"/>
                 </geometry>
             </collision>
@@ -135,5 +135,5 @@
                 <origin xyz="0 0 0" rpy="0 0 0"/>
                 <geometry>
-                    <mesh filename="file://$(find smb_description)/urdf/meshes/SMB_step.dae"/>
+                    <mesh filename="package://smb_description/urdf/meshes/SMB_step.dae"/>
                 </geometry>
             </visual>

File: urdf/smb_lidar_mount.urdf.xacro (robot description, xacro)
@@ -12,5 +12,5 @@
       <visual>
         <geometry>
-          <mesh filename="file://$(find smb_description)/urdf/meshes/LidarBoxV2.dae"/>
+          <mesh filename="package://smb_description/urdf/meshes/LidarBoxV2.dae"/>
         </geometry>
       </visual>
